File: PiPicoOssciloscope_THT/Input.kicad_sch (KiCad schematic)
At the start: 83 parts, among them J1 Conn_Coaxial, J2 Conn_Coaxial, U1 SMQS-04R-TP, U2 SMQS-04R-TP, U3 SMQS-04R-TP, U4 SMQS-04R-TP, U5 SMQS-04R-TP, U6 SMQS-04R-TP, U7 SMQS-04R-TP, U8 MCP6002-I/P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

Commit message: updated the bnc connector
Parts:
- J1, J2: footprint Connector_Coaxial:BNC_TEConnectivity_1478035_Horizontal -> Connector_Coaxial:BNC_Amphenol_B6252HB-NPP3G-50_Horizontal
Changed lines of the file:
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@@
 			)
 		)
-		(property "Footprint" "Connector_Coaxial:BNC_TEConnectivity_1478035_Horizontal"
+		(property "Footprint" "Connector_Coaxial:BNC_Amphenol_B6252HB-NPP3G-50_Horizontal"
 			(at 57.15 24.13 0)
 			(hide yes)
@@
 			)
 		)
-		(property "Footprint" "Connector_Coaxial:BNC_TEConnectivity_1478035_Horizontal"
+		(property "Footprint" "Connector_Coaxial:BNC_Amphenol_B6252HB-NPP3G-50_Horizontal"
 			(at 31.75 24.13 0)
 			(hide yes)
